Commit message: for the pneumatic flange this is needed, tested on the robot

File: urdf/iiwa14.xacro (robot description, xacro)
@@ -307,4 +307,11 @@
     <link name="${robot_name}_link_ee_kuka">
     </link>
+    <joint name="${robot_name}_joint_ee_pneumatic" type="fixed">
+      <parent link="${robot_name}_link_ee_kuka"/>
+      <child link="${robot_name}_link_ee_pneumatic"/>
+      <origin xyz="0 0 0.026" rpy="0 0 0"/>
+    </joint>
+    <link name="${robot_name}_link_ee_pneumatic">
+    </link>
     <!--Extensions -->
     <xacro:iiwa_gazebo robot_name="${robot_name}" />
